File: H1FR50/Design/H1FR50.sch (EAGLE design)
At the start: 34 parts, among them P2 HEXABIT_X2_P1_P5, Q1 MMBT3904LT1, Q2 MMBT3904LT1, U1 STM32G0B1CEU6NUFQFPN48_STM32_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, U2 SAM-M8Q-0-10

Commit message: -Update the GNSS Module (SAM-M10Q-00B) in BOM and Schematic files
Parts:
- U2: MP (none) -> SAM-M10Q-00B
Changed lines of the file:
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@@
 <?xml version="1.0" encoding="utf-8"?>
 <!DOCTYPE eagle SYSTEM "eagle.dtd">
-<eagle version="9.6.1">
+<eagle version="9.6.2">
 <drawing>
 <settings>
@@
 <part name="SUPPLY9" library="supply2" deviceset="VDD" device=""/>
 <part name="JP2" library="pinhead" deviceset="PINHD-1X3" device="" package3d_urn="urn:adsk.eagle:package:22458/2"/>
-<part name="U2" library="SAM-M8Q-0-10" deviceset="SAM-M8Q-0-10" device="" override_package3d_urn="urn:adsk.eagle:package:37789442/2" override_package_urn="urn:adsk.eagle:footprint:37789443/1"/>
+<part name="U2" library="SAM-M8Q-0-10" deviceset="SAM-M8Q-0-10" device="" override_package3d_urn="urn:adsk.eagle:package:37789442/2" override_package_urn="urn:adsk.eagle:footprint:37789443/1">
+<attribute name="MP" value="SAM-M10Q-00B"/>
+</part>
 <part name="SUPPLY5" library="supply2" deviceset="VDD" device=""/>
 <part name="GND4" library="supply1" library_urn="urn:adsk.eagle:library:371" deviceset="GND" device=""/>
@@
 <instance part="U2" gate="G$1" x="184.15" y="107.95" smashed="yes">
 <attribute name="NAME" x="168.91" y="124.079" size="1.778" layer="95"/>
-<attribute name="VALUE" x="168.91" y="90.17" size="1.778" layer="96"/>
+<attribute name="MP" x="168.91" y="90.17" size="1.778" layer="96"/>
 </instance>
 <instance part="SUPPLY5" gate="G$1" x="212.09" y="128.27" smashed="yes">
